File: PCB/Stemma_Host_FeatherWing.sch (KiCad schematic (older format))
At the start: 15 parts, among them J1 STEMMA, J2 STEMMA, J3 STEMMA-QT, J4 STEMMA-QT, M1 Feather_M4_Express, U1 BSS138DW-Y-F_ALT, U2 AP2112-3.3

Commit message: update with initial design
Parts:
- removed C2: 0.1uF, Capacitors_SMD:C_0805, symbol device:C_Small
- removed C3: 10uF, Capacitors_SMD:C_0805, symbol device:CP1_Small
- removed U2: AP2112-3.3, TO_SOT_Packages_SMD:SOT-23-5, symbol regul:AP2112-3.3
- added D2, D3: MBR120, Diodes_SMD:D_SOD-123F, symbol device:D_Schottky_Small
- added SW1: SW_Push, Adafruit:TL3330AF_SPST_BUTTON_RT-ANGLE_7.8mm_2.5mm_2.5mm, symbol switches:SW_Push
Connections:
- wire segments 141 -> 128
- no-connect marks 22 -> 19
Other:
- note removed: "POWER MGT"

Commit message: update design
Parts:
- added JMP3: STEMMA_TYPE, Connectors:GS3, symbol conn:GS3
Connections:
- wire segments 128 -> 132
Changed lines of the file:
@@
 Wire Wire Line
 	2950 2650 2975 2650
-Text Label 6400 800  0    50   ~ 0
+Text Label 7550 900  0    50   ~ 0
 +V
 $Comp
@@
 FEATHER PINS
 Wire Wire Line
-	6400 800  6400 1225
+	7550 900  7550 1325
 Connection ~ 6400 2375
 Wire Wire Line
 	6400 1225 6400 2375
-Connection ~ 6400 1225
 Wire Wire Line
 	2550 2550 2550 2475
@@
 Wire Wire Line
 	5175 5450 7025 5450
+$Comp
+L conn:GS3 JMP3
+U 1 1 5DDE749D
+P 7100 1225
+F 0 "JMP3" H 7100 950 50  0000 C CNN
+F 1 "STEMMA_TYPE" H 7100 1025 50  0000 C CNN
+F 2 "Connectors:GS3" V 7188 1151 50  0001 C CNN
+F 3 "" H 7100 1225 50  0001 C CNN
+	1    7100 1225
+	-1   0    0    -1
+$EndComp
+$Comp
+L power:+3.3V #PWR0110
+U 1 1 5DDF140E
+P 7350 1000
+F 0 "#PWR0110" H 7350 850 50  0001 C CNN
+F 1 "+3.3V" H 7365 1173 50  0000 C CNN
+F 2 "" H 7350 1000 50  0001 C CNN
+F 3 "" H 7350 1000 50  0001 C CNN
+	1    7350 1000
+	1    0    0    -1
+$EndComp
+Wire Wire Line
+	6400 1225 6950 1225
+Connection ~ 6400 1225
+Wire Wire Line
+	7250 1125 7350 1125
+Wire Wire Line
+	7350 1000 7350 1125
+Wire Wire Line
+	7250 1325 7550 1325
 $EndSCHEMATC

Commit message: initial repo load
Connections:
- wire segments 132 -> 137
Other:
- note added: "~~5V"
- note added: "~~5V default jumper"
Changed lines of the file:
@@
 U 1 1 5DDE749D
 P 7100 1225
-F 0 "JMP3" H 7100 950 50  0000 C CNN
-F 1 "STEMMA_TYPE" H 7100 1025 50  0000 C CNN
+F 0 "JMP3" H 7125 1500 50  0000 C CNN
+F 1 "STEMMA_TYPE" H 7275 1425 50  0000 C CNN
 F 2 "Connectors:GS3" V 7188 1151 50  0001 C CNN
 F 3 "" H 7100 1225 50  0001 C CNN
@@
 $EndComp
 Wire Wire Line
-	6400 1225 6950 1225
+	6400 1225 6875 1225
 Connection ~ 6400 1225
 Wire Wire Line
@@
 	7350 1000 7350 1125
 Wire Wire Line
-	7250 1325 7550 1325
+	7250 1325 7325 1325
+Wire Wire Line
+	6875 1225 6875 1450
+Wire Wire Line
+	6875 1450 7325 1450
+Wire Wire Line
+	7325 1450 7325 1325
+Connection ~ 6875 1225
+Wire Wire Line
+	6875 1225 6950 1225
+Connection ~ 7325 1325
+Wire Wire Line
+	7325 1325 7550 1325
+Text Notes 7375 1300 0    50   ~ 0
+~~5V
+Text Notes 7375 1525 0    50   ~ 0
+~~5V default jumper
 $EndSCHEMATC

Commit message: PCB version update
Parts:
- U1: value BSS138DW-Y-F_ALT -> BSS138DW/BK; footprint TO_SOT_Packages_SMD:SOT-23-6 -> TO_SOT_Packages_SMD:SOT-363_SC-70-6
Changed lines of the file:
@@
 Sheet 1 1
 Title "Stemma_Host_FeatherWing"
-Date "2019-11-25"
-Rev "v01"
+Date "2019-12-09"
+Rev "v02"
 Comp "Cedar Grove Studios"
 Comment1 ""
@@
 P 4550 2925
 F 0 "U1" H 4550 2303 50  0000 C CNN
-F 1 "BSS138DW-Y-F_ALT" H 4550 2212 50  0000 C CNN
-F 2 "TO_SOT_Packages_SMD:SOT-23-6" H 4550 2925 50  0001 C CNN
+F 1 "BSS138DW/BK" H 4550 2212 50  0000 C CNN
+F 2 "TO_SOT_Packages_SMD:SOT-363_SC-70-6" H 4550 2925 50  0001 C CNN
 F 3 "" H 4550 2925 50  0001 C CNN
 	1    4550 2925
